File: kicad/ITX-Llama.kicad_sch (KiCad schematic)
At the start: 421 parts, among them J1 ATX_POWER, J10 SATA, J11 SPEAKER, J12 MSD, J14 AUDIO, J15 KBC, J16 KBD, J17 USB_ETH, J18 USB_HID, J19 HID_POWER, J2 MICRO_SD, J20 FAN1, J21 FAN2, J22 GAMEPORT, J23 WAVETABLE, J24 PI_ZERO2, J25 POWER, J26 LEFT, J27 RIGHT, J28 COM2_TTL, J29 PI_2/3/4, J3 FRONT_PANEL, J30 FAN3, J31 FAN1_VDD, J32 FAN2_VDD, J33 FAN3_VDD, J34 CD_IN, J35 D1_MINI, J36 ESP_POWER, J38 J_TOSLINK_ZGY133T10, J39 LINE_L, J4 PS/2, J40 LINE_R, J41 EXT_SYNTH, J42 PI_I2C, J43 I2C, J46 RP_DEBUG, J5 AGP_3.3V, J6 CLICK_VOL, J7 MSC, J8 COM1, J9 INT_SPKR_VOL, P1 P_SOM-128-EX, Q1 NPN, Q10 Q_NMOS_GDS, Q11 Q_NMOS_GDS, Q2 NPN, Q3 NPN, Q4 NPN, Q5 NPN, Q6 NPN, Q7 NPN, Q8 Q_NMOS_GDS, Q9 Q_NMOS_GDS, SW1 CH559_PRG, SW1 POWER, SW2 RESET, T1 Pulse_H1102NL, U1 MAX16054, U10 U_MIC5219-3.3YM5, U11 EMC2303, U12 PCM5102A, U13 U_MIC5219-3.3YM5, U14 U_MIC5219-3.3YM5, U15 W25Q32JVSS, U16 U_74LVC1G126, U17 U_RP2040, U2 U_74LVC1G04, U3 U_CS4237B-KQ, U4 GD75232, U5 U_MC33078, U6 PI7C9X118SL, U7 AP7165, U8 U_MIC5219-3.3YM5, U9 U_ATTINY84A, X1 16.9344MHz, X2 12MHz

Commit message: revK
Parts:
- C100, C101, C102, C103, C104, C105, C106, C107, C108, C109, C110, C111, C112, C113, C114, C115, C116, C117, C118, C119, C12, C120, C121, C122, C123, C124, C125, C126, C127, C128, C129, C13, C130, C131, C132, C133, C135, C136, C138, C14, C141, C142, C144, C145, C146, C15, C150, C151, C152, C153, C156, C157, C16, C160, C162, C163, C164, C165, C166, C17, C177, C178, C179, C18, C180, C181, C182, C183, C184, C185, C186, C187, C188, C189, C19, C190, C20, C21, C22, C23, C24, C25, C26, C28, C29, C35, C36, C37, C38, C39, C40, C41, C42, C51, C54, C55, C56, C57, C58, C59, C6, C60, C63, C64, C65, C66, C67, C7, C70, C71, C72, C73, C78, C79, C8, C84, C85, C86, C87, C89, C90, C91, C92, C93, C94, C95, C96, C97, C98, C99: footprint llama_shared:C_0402_1005Metric -> llama_shared:C_0603_1608Metric
- C48, C49, C50, C81, C82, C83: renamed from C1; footprint llama_shared:C_0402_1005Metric -> llama_shared:C_0603_1608Metric
- FB1, FB2, R1, R10, R100, R101, R102, R103, R104, R105, R106, R107, R108, R109, R11, R110, R111, R112, R113, R114, R115, R116, R117, R118, R119, R12, R120, R121, R13, R14, R17, R18, R19, R2, R20, R21, R22, R23, R24, R25, R26, R27, R28, R29, R3, R30, R31, R32, R33, R34, R35, R36, R37, R38, R39, R4, R40, R41, R42, R43, R44, R45, R46, R47, R48, R49, R5, R50, R51, R52, R53, R54, R55, R56, R57, R58, R6, R60, R61, R62, R63, R64, R65, R68, R69, R7, R70, R71, R72, R73, R74, R75, R76, R77, R78, R79, R8, R80, R81, R82, R83, R84, R85, R86, R87, R88, R89, R9, R90, R91, R92, R93, R97, R98, R99: footprint llama_shared:R_0402_1005Metric -> llama_shared:R_0603_1608Metric
- R15: renamed from R1; footprint llama_shared:R_0402_1005Metric -> llama_shared:R_0603_1608Metric
- R16: renamed from R2; footprint llama_shared:R_0402_1005Metric -> llama_shared:R_0603_1608Metric
- R66: renamed from R3; footprint llama_shared:R_0402_1005Metric -> llama_shared:R_0603_1608Metric
- R67: renamed from R4; footprint llama_shared:R_0402_1005Metric -> llama_shared:R_0603_1608Metric
- renumbered C1 to C80, SW1 to SW3
